File: csa_ultrabus_v2.brd (EAGLE design)
At the start: 160 x 100 mm, 59 parts, among them IC1 74AC04D, IC2 74AC138D, IC3 74AC138D, IC4 74AC138D, IC5 74AC138D, IC6 74HCT00D, IC7 74HCT125D, IC8 74HCT125D, P1 CSABUS, P2 CSABUSSOCK180, P3 CSABUSSOCK180, P4 CSABUSSOCK180

Commit message: revision 2.0b
Parts:
- removed JP3, JP4, JP5, JP6, JP7: (no value), jumper:JP2
- removed SLOT6.3: RC2014/650239+1R, csa:SIL39+1R
- added C22: (no value), rcl:C0603
- added C23, C24: 47u, rcl:E2,5-5
- added IC9: 74AC138D, 74xx-eu:SO16
- added U$1: CSASHORTBUSFS, csa:FABC48S2
- added U$2: CSASHORTBUSMA, csa:MABC48B2
- added X1: PORT_EXPANSION_64_CONN, commodore:FE100-22-2
- P1: value CSABUS -> CSABUSSOCK180; device csa:CSABUS -> csa:CSABUSSOCK180
- SLOT6.1, SLOT6.2: value RC2014/650239+1R -> RC2014/6502; device csa:SIL39+1R -> csa:SIL40
- moved JP2 42.8 mm to (150.2, 4.29)
- moved C18 33.4 mm to (149.1, 8.57), turned to 180 degrees
- moved P1 10.5 mm to (3.10, 52.1)
- moved SLOT6.1 6.60 mm to (123.0, 29.3)
- moved SLOT6.2 6.53 mm to (137.9, 29.1)
Connections:
- removed net /BANK4_Q: IC6.8, SLOT6.1.23
- removed net /SEL6: IC1.11, JP14.2, JP3.3, SLOT6.2.23
- removed net /SLOT4IO_Q: IC6.11, SLOT6.1.26
- removed net 8PHI2: P1.C31, P2.C31, P3.C31, P4.C31
- removed net N$10: JP7.2, SLOT6.3.37
- removed net N$2: JP3.2, SLOT6.3.23
- removed net N$4: JP4.2, SLOT6.3.24
- new net /BANK1: IC2.14, JP2.1
- new net /BANK3: IC2.12, JP2.3
- new net /SLOT1IO: IC3.14, X1.7
- new net /SLOT4IO: IC3.11, X1.10
- new net /SLOT6.X_BANK: IC6.8, SLOT6.1.23, SLOT6.2.23
- new net /SLOT6.X_IO: IC6.11, SLOT6.1.26, SLOT6.2.26
- new net N$23: IC9.4, JP2.2
- new net RC_CLK: SLOT6.1.21, SLOT6.2.21
- net /BE: now also U$1.A4, U$2.A4
- net /IOSEL: now also U$1.A3, U$2.A3
- net /IRQ: now also U$1.A14, U$2.A14, X1.4; no longer SLOT6.3.22
- net /M1: no longer JP2.3
- net /MEMSEL: now also U$1.A2, U$2.A2
- net /NMI: now also U$1.A13, U$2.A13, X1.D; no longer JP7.1
- net /RD0: no longer JP5.3
- net /RES: now also U$1.A15, U$2.A15, X1.C; no longer SLOT6.3.20
- net /SLOT6IO: no longer JP6.3, SLOT6.2.26
- net /WR0: no longer JP4.3
- net B2PHI2: now also U$1.C15, U$2.C15
- net B8PHI2: now also P1.C31, P2.C31, P3.C31, P4.C31, U$1.B16, U$2.B16, X1.6
- net BA0: now also U$1.C11, U$2.C11, X1.Y; no longer SLOT6.3.16
- net BA1: now also U$1.B10, U$2.B10, X1.X; no longer SLOT6.3.15
- net BA10: now also U$1.C6, U$2.C6, X1.M; no longer SLOT6.3.6
- net BA11: now also U$1.B5, U$2.B5, X1.L; no longer SLOT6.3.5
- net BA12: now also U$1.C5, U$2.C5, X1.K; no longer SLOT6.3.4
- net BA13: now also IC9.1, U$1.B4, U$2.B4, X1.J; no longer SLOT6.3.3
- net BA14: now also IC9.2, U$1.C4, U$2.C4, X1.H; no longer SLOT6.3.2
- net BA15: now also IC9.3, U$1.B3, U$2.B3, X1.F; no longer SLOT6.3.1
- net BA16: now also U$1.C3, U$2.C3
- net BA17: now also U$1.B2, U$2.B2
- net BA18: now also U$1.C2, U$2.C2
- net BA19: now also U$1.B1, U$2.B1
- net BA2: now also U$1.C10, U$2.C10, X1.W; no longer SLOT6.3.14
- net BA3: now also U$1.B9, U$2.B9, X1.V; no longer SLOT6.3.13
- net BA4: now also U$1.C9, U$2.C9, X1.U; no longer SLOT6.3.12
- net BA5: now also U$1.B8, U$2.B8, X1.T; no longer SLOT6.3.11
- net BA6: now also U$1.C8, U$2.C8, X1.S; no longer SLOT6.3.10
- net BA7: now also U$1.B7, U$2.B7, X1.R; no longer SLOT6.3.9
- net BA8: now also U$1.C7, U$2.C7, X1.P; no longer SLOT6.3.8
- net BA9: now also U$1.B6, U$2.B6, X1.N; no longer SLOT6.3.7
- net BD0: now also U$1.A12, U$2.A12, X1.21; no longer SLOT6.3.27
- net BD1: now also U$1.A11, U$2.A11, X1.20; no longer SLOT6.3.28
- net BD2: now also U$1.A10, U$2.A10, X1.19; no longer SLOT6.3.29
- net BD3: now also U$1.A9, U$2.A9, X1.18; no longer SLOT6.3.30
- net BD4: now also U$1.A8, U$2.A8, X1.17; no longer SLOT6.3.31
- net BD5: now also U$1.A7, U$2.A7, X1.16; no longer SLOT6.3.32
- net BD6: now also U$1.A6, U$2.A6, X1.15; no longer SLOT6.3.33
- net BD7: now also U$1.A5, U$2.A5, X1.14; no longer SLOT6.3.34
- net BPHI0: now also U$1.C14, U$2.C14; no longer SLOT6.1.21, SLOT6.2.21, SLOT6.3.21
- net BPHI1: now also U$1.C13, U$2.C13; no longer JP3.1
- net BPHI2: now also IC6.12, IC6.9, U$1.C12, U$2.C12, X1.E; no longer JP2.1
- net GND: now also C22.2, C23.-, C24.-, IC9.5, IC9.8, U$1.A1, U$1.A16, U$2.A1, U$2.A16, X1.1, X1.22, X1.A, X1.Z; no longer SLOT6.3.17
- net N$1: now also IC1.11, JP14.2; no longer JP2.2, SLOT6.3.19
- net N$6: now also IC9.7, X1.B; no longer JP5.2, SLOT6.3.25
- net N$7: now also IC9.11, X1.11; no longer JP6.2, SLOT6.3.26
- net R/-W: now also U$1.B12, U$2.B12, X1.5; no longer IC6.12, IC6.9, JP4.1
- net RDY: now also U$1.B13, U$2.B13; no longer JP5.1
- net RX: no longer SLOT6.3.36
- net SYNC: now also U$1.B11, U$2.B11; no longer JP6.1
- net TX: no longer SLOT6.3.35
- net USER1: no longer JP7.3
- net USER2: no longer SLOT6.3.38
- net USER3: no longer SLOT6.3.39
- net USER4: no longer SLOT6.3.40
- net VBUF: now also U$1.B15, U$2.B15
- net VCC: now also C22.1, C23.+, C24.+, IC9.16, IC9.6, U$1.C1, U$1.C16, U$2.C1, U$2.C16, X1.2, X1.3; no longer SLOT6.3.18
- net VCC33: now also U$1.B14, U$2.B14
Routing:
- net B8PHI2: track 0.00 -> 220.5 mm, vias 0 -> 5
- net /SLOT4IO: track 0.00 -> 194.0 mm, vias 0 -> 5
- net /SLOT1IO: track 0.00 -> 170.5 mm, vias 0 -> 3
- net /SEL6: track 169.7 -> 0.00 mm, vias 7 -> 0
- net BPHI0: track 189.8 -> 58.1 mm, vias 2 -> 0
- net /BANK3: track 0.00 -> 115.5 mm, vias 0 -> 5
- net /SLOT6IO: track 182.6 -> 80.5 mm, vias 6 -> 2
- net N$23: track 0.00 -> 100.4 mm, vias 0 -> 2
- net /BANK1: track 0.00 -> 95.7 mm, vias 0 -> 5
- net N$1: track 9.94 -> 102.5 mm, vias 1 -> 4
- net BA13: track 192.5 -> 283.4 mm, vias 2 -> 3
- net GND: track 1034.5 -> 1124.5 mm, vias 21 -> 25
- net VCC: track 824.9 -> 906.0 mm, vias 16 -> 18
- net RDY: track 251.6 -> 176.3 mm, vias 4 -> 3
- net BA14: track 210.7 -> 281.7 mm
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Other:
- board text added: "CSA-ULTRABUS-V1.1A (C) A. Fachat"
- board text removed: "RC2014"
- board text removed: "RC2014 / RC6502 Combi"
- board text removed: "RC6502"
- board text removed: "SLOT6.3 MODE"
