File: csa_ultrabus_v2.sch (EAGLE design)
At the start: 59 parts, among them IC1 74AC04D, IC2 74AC138D, IC3 74AC138D, IC4 74AC138D, IC5 74AC138D, IC6 74HCT00D, IC7 74HCT125D, IC8 74HCT125D, P1 CSABUS, P2 CSABUSSOCK180, P3 CSABUSSOCK180, P4 CSABUSSOCK180

Commit message: revision 2.0b
Parts:
- removed JP3, JP4, JP5, JP6, JP7: (no value), jumper:JP2E
- removed SLOT6.3: RC2014/650239+1R, csa:RC2014/650239+1R
- added C22: (no value), rcl:C-EUC0603
- added C23, C24: 47u, rcl:CPOL-EUE2.5-5
- added IC9: 74AC138D, 74xx-eu:74AC138D
- added U$1: CSASHORTBUSFS, csa:CSASHORTBUSFS
- added U$2: CSASHORTBUSMA, csa:CSASHORTBUSMA
- added X1: PORT_EXPANSION_64_CONN, commodore:PORT_EXPANSION_64_CONN
- P1: value CSABUS -> CSABUSSOCK180; device csa:CSABUS -> csa:CSABUSSOCK180
- SLOT6.1, SLOT6.2: value RC2014/650239+1R -> RC2014/6502; device csa:RC2014/650239+1R -> csa:RC2014/6502
Connections:
- removed net /BANK4_Q: IC6C.O, SLOT6.1.*PHI1,/MREQ
- removed net /SEL6: IC1E.I, JP14.2, JP3.3, SLOT6.2.*PHI1,/MREQ
- removed net /SLOT4IO_Q: IC6D.O, SLOT6.1.*SYNC,/IOREQ
- removed net 8PHI2: P1.8PHI2, P2.8PHI2, P3.8PHI2, P4.8PHI2
- removed net N$10: JP7.2, SLOT6.3.*/NMI,USER1
- removed net N$2: JP3.2, SLOT6.3.*PHI1,/MREQ
- removed net N$4: JP4.2, SLOT6.3.*R/-W,/WR
- new net /BANK1: IC2A.Y1, JP2.1
- new net /BANK3: IC2A.Y3, JP2.3
- new net /SLOT1IO: IC3A.Y1, X1A.!IO1
- new net /SLOT4IO: IC3A.Y4, X1A.!IO2
- new net /SLOT6.X_BANK: IC6C.O, SLOT6.1.*PHI1,/MREQ, SLOT6.2.*PHI1,/MREQ
- new net /SLOT6.X_IO: IC6D.O, SLOT6.1.*SYNC,/IOREQ, SLOT6.2.*SYNC,/IOREQ
- new net N$23: IC9A.G2A, JP2.2
- new net RC_CLK: SLOT6.1.PHI0,CLK, SLOT6.2.PHI0,CLK
- net /BE: now also U$1./BE, U$2./BE
- net /IOSEL: now also U$1./IOSEL, U$2./IOSEL
- net /IRQ: now also U$1./IRQ, U$2./IRQ, X1A.!IRQ; no longer SLOT6.3./IRQ
- net /M1: no longer JP2.3
- net /MEMSEL: now also U$1./MEMSEL, U$2./MEMSEL
- net /NMI: now also U$1./NMI, U$2./NMI, X1A.!NMI; no longer JP7.1
- net /RD0: no longer JP5.3
- net /RES: now also U$1./RES, U$2./RES, X1A.!RESET; no longer SLOT6.3./RES
- net /SLOT6IO: no longer JP6.3, SLOT6.2.*SYNC,/IOREQ
- net /WR0: no longer JP4.3
- net B2PHI2: now also U$1.2PHI2, U$2.2PHI2
- net B8PHI2: now also P1.8PHI2, P2.8PHI2, P3.8PHI2, P4.8PHI2, U$1.8PHI2, U$2.8PHI2, X1A.DOTCLK
- net BA0: now also U$1.A0, U$2.A0, X1A.A0; no longer SLOT6.3.A0
- net BA1: now also U$1.A1, U$2.A1, X1A.A1; no longer SLOT6.3.A1
- net BA10: now also U$1.A10, U$2.A10, X1A.A10; no longer SLOT6.3.A10
- net BA11: now also U$1.A11, U$2.A11, X1A.A11; no longer SLOT6.3.A11
- net BA12: now also U$1.A12, U$2.A12, X1A.A12; no longer SLOT6.3.A12
- net BA13: now also IC9A.A, U$1.A13, U$2.A13, X1A.A13; no longer SLOT6.3.A13
- net BA14: now also IC9A.B, U$1.A14, U$2.A14, X1A.A14; no longer SLOT6.3.A14
- net BA15: now also IC9A.C, U$1.A15, U$2.A15, X1A.A15; no longer SLOT6.3.A15
- net BA16: now also U$1.A16, U$2.A16
- net BA17: now also U$1.A17, U$2.A17
- net BA18: now also U$1.A18, U$2.A18
- net BA19: now also U$1.A19, U$2.A19
- net BA2: now also U$1.A2, U$2.A2, X1A.A2; no longer SLOT6.3.A2
- net BA3: now also U$1.A3, U$2.A3, X1A.A3; no longer SLOT6.3.A3
- net BA4: now also U$1.A4, U$2.A4, X1A.A4; no longer SLOT6.3.A4
- net BA5: now also U$1.A5, U$2.A5, X1A.A5; no longer SLOT6.3.A5
- net BA6: now also U$1.A6, U$2.A6, X1A.A6; no longer SLOT6.3.A6
- net BA7: now also U$1.A7, U$2.A7, X1A.A7; no longer SLOT6.3.A7
- net BA8: now also U$1.A8, U$2.A8, X1A.A8; no longer SLOT6.3.A8
- net BA9: now also U$1.A9, U$2.A9, X1A.A9; no longer SLOT6.3.A9
- net BD0: now also U$1.D0, U$2.D0, X1A.D0; no longer SLOT6.3.D0
- net BD1: now also U$1.D1, U$2.D1, X1A.D1; no longer SLOT6.3.D1
- net BD2: now also U$1.D2, U$2.D2, X1A.D2; no longer SLOT6.3.D2
- net BD3: now also U$1.D3, U$2.D3, X1A.D3; no longer SLOT6.3.D3
- net BD4: now also U$1.D4, U$2.D4, X1A.D4; no longer SLOT6.3.D4
- net BD5: now also U$1.D5, U$2.D5, X1A.D5; no longer SLOT6.3.D5
- net BD6: now also U$1.D6, U$2.D6, X1A.D6; no longer SLOT6.3.D6
- net BD7: now also U$1.D7, U$2.D7, X1A.D7; no longer SLOT6.3.D7
- net BPHI0: now also U$1.PHI0, U$2.PHI0; no longer SLOT6.1.PHI0,CLK, SLOT6.2.PHI0,CLK, SLOT6.3.PHI0,CLK
- net BPHI1: now also U$1.PHI1, U$2.PHI1; no longer JP3.1
- net BPHI2: now also IC6C.I0, IC6D.I0, U$1.PHI2, U$2.PHI2, X1A.PHI2; no longer JP2.1
- net GND: now also C22.2, C23.-, C24.-, IC9A.G2B, U$1.GND, U$1.GND2, U$2.GND, U$2.GND2, X1P.GND, X1P.GND@1, X1P.GND@2, X1P.GND@3; no longer SLOT6.3.GND
- net N$1: now also IC1E.I, JP14.2; no longer JP2.2, SLOT6.3.*PHI2,/M1
- net N$6: now also IC9A.Y7, X1A.!ROMH; no longer JP5.2, SLOT6.3.*RDY,/RD
- net N$7: now also IC9A.Y4, X1A.!ROML; no longer JP6.2, SLOT6.3.*SYNC,/IOREQ
- net R/-W: now also U$1.R/-W, U$2.R/-W, X1A.R/!W; no longer IC6C.I0, IC6D.I0, JP4.1
- net RDY: now also U$1.RDY, U$2.RDY; no longer JP5.1
- net RX: no longer SLOT6.3.RX
- net SYNC: now also U$1.SYNC, U$2.SYNC; no longer JP6.1
- net TX: no longer SLOT6.3.TX
- net USER1: no longer JP7.3
- net USER2: no longer SLOT6.3.EX1/USER2
- net USER3: no longer SLOT6.3.EX2/USER3
- net USER4: no longer SLOT6.3.USER4
- net VBUF: now also U$1.VBUF, U$2.VBUF
- net VCC: now also C22.1, C23.+, C24.+, IC9A.G1, U$1.VCC, U$1.VCC2, U$2.VCC, U$2.VCC2, X1P.VCC, X1P.VCC@1; no longer SLOT6.3.VCC
- net VCC33: now also U$1.VCC33, U$2.VCC33
Other:
- note added: "$C1xx"
- note added: "$C2xx"
- note added: "$C3xx"
- note added: "$C4xx"
- note added: "$C5xx"
- note added: "$C6xx"
- note added: "1.0B: - fix qualifying SLOTIO and BANK with Phi2 - separate RC_CLK from BPHI0 1.1A: - remove RC6502 slot - Both remaining RC2014 now have MREQ and IOREQ qualified with Phi2"
- note added: "CS/A65 Ultra BUS 1.1A"
- note added: "CSA-ULTRABUS-V1.1A-20240215"
- note removed: "CS/A65 Ultra BUS"
- note removed: "Only slot with /MEMRQ and /IORQ qualified with PHI2 (e.g. needed by 6850 based serial RC2014 card)"
