File: Board/csa_ultrabus_v2.kicad_sch (KiCad schematic)
At the start: 0 parts

Commit message: layout ubus 2.1a
Other:
- added sheet usbpd (usbpd.kicad_sch)
- added sheet usbpd control LEDs (usbpd_leds.kicad_sch)
- added sheet usbpd negative voltages (usbpd_neg.kicad_sch)
- added sheet usbpd positive voltages (usbpd_pos.kicad_sch)
- note added: "(C) A. Fachat"
- note added: "2.0A: - add shortbus connector as extension of the UltiPET 2.0B: - Add pullup on JP9 2.1A: - replace power connector with USB-C based power converters"
- note added: "CS/A65 Ultra BUS 2.1A"
- note added: "CSA-ULTRABUS-V2.0B-20240523"
