File: Board/Apple_II_Bus.kicad_sch (KiCad schematic)
At the start: 34 parts, among them IC1 7404D, IC2 74138D, IC3 74138D, IC4 74138D, IC5 74138D, IC6 7400D, IC7 74125D, IC8 74125D, IC9 74138D

Commit message: layout ubus 2.1a
Connections:
- net -5V: now reaches SLOT5.R (-5V)
- net -5V: now also SLOT3.R (-5V), SLOT7.R (-5V)
- net -12V: now reaches SLOT5.S (-12V)
- net -12V: now also SLOT3.S (-12V), SLOT7.S (-12V)
Other:
- note added: "CS/A65 Ultra BUS 2.1A"
- note removed: "CS/A65 Ultra BUS 2.0B"

Commit message: candidate
Parts:
- C10, C11, C12, C16, C2, C7, C8, C9: LCSC (none) -> C14663
- C13, C14, C15, C19, C20, C21: LCSC (none) -> C713185
- IC1: LCSC (none) -> C6766
- IC2, IC3, IC4, IC5, IC9: LCSC (none) -> C352958
- IC6: LCSC (none) -> C282337
- IC7, IC8: LCSC (none) -> C5962
- JP10, JP11, JP15, JP16, JP9: LCSC (none) -> C6332196
- JP17, JP8: LCSC (none) -> C7494857
- R1: footprint Resistor_THT:R_Axial_DIN0204_L3.6mm_D1.6mm_P2.54mm_Vertical -> Resistor_SMD:R_0603_1608Metric_Pad0.98x0.95mm_HandSolder; LCSC (none) -> C25804
- SLOT3, SLOT5, SLOT7: LCSC (none) -> C5173308
