File: Board/C64.kicad_sch (KiCad schematic)
At the start: 4 parts, among them IC9 74138D, X1 PORT_EXPANSION_64_CONN

Commit message: layout ubus 2.1a
Other:
- note added: "CS/A65 Ultra BUS 2.1A"
- note removed: "CS/A65 Ultra BUS 2.0B"

Commit message: candidate
Parts:
- C22: LCSC (none) -> C14663
- IC9: LCSC (none) -> C352958
- JP2: LCSC (none) -> C6332196
- X1: LCSC (none) -> C21261712
Changed lines of the file:
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@@
+			)
+		)
+		(property "LCSC" "C21261712"
+			(at 139.7 88.9 0)
+			(effects
+				(font
+					(size 1.27 1.27)
+				)
+				(hide yes)
 			)
 		)
@@
 			)
 		)
+		(property "LCSC" "C21261712"
+			(at 66.04 101.6 0)
+			(effects
+				(font
+					(size 1.27 1.27)
+				)
+				(hide yes)
+			)
+		)
 		(pin "10"
 		)
@@
 			)
 		)
+		(property "LCSC" "C6332196"
+			(at 163.83 144.78 0)
+			(effects
+				(font
+					(size 1.27 1.27)
+				)
+				(hide yes)
+			)
+		)
 		(pin "1"
 		)
@@
 			)
 		)
+		(property "LCSC" "C352958"
+			(at 210.185 142.875 0)
+			(effects
+				(font
+					(size 1.27 1.27)
+				)
+				(hide yes)
+			)
+		)
 		(pin "1"
 		)
@@
 			)
 		)
+		(property "LCSC" "C14663"
+			(at 82.804 98.679 0)
+			(effects
+				(font
+					(size 1.27 1.27)
+				)
+				(hide yes)
+			)
+		)
