File: Board/CS%2fA_BUS.kicad_sch (KiCad schematic)
At the start: 19 parts, among them J1 FLOP-4W827001, P1 CSABUSSOCK180, P2 CSABUSSOCK180, P3 CSABUSSOCK180, P4 CSABUSSOCK180

Commit message: layout ubus 2.1a
Parts:
- removed J1: FLOP-4W827001, csa_ultrabus_v2:827001, symbol csa_ultrabus_v2-eagle-import:FLOP-4W827001
Other:
- note added: "CS/A65 Ultra BUS 2.1A"
- note removed: "CS/A65 Ultra BUS 2.0B"

Commit message: candidate
Parts:
- C1, C17, C18, C3, C4, C5, C6: LCSC (none) -> C713185
- JP1: LCSC (none) -> C6332196
- P1, P2, P3, P4: LCSC (none) -> C53202145
Changed lines of the file:
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@@
+			)
+		)
+		(property "LCSC" "C713185"
+			(at 453.263 85.8774 0)
+			(effects
+				(font
+					(size 1.27 1.27)
+				)
+				(hide yes)
 			)
 		)
@@
 			)
 		)
+		(property "LCSC" "C713185"
+			(at 44.323 164.6174 0)
+			(effects
+				(font
+					(size 1.27 1.27)
+				)
+				(hide yes)
+			)
+		)
 		(pin "+"
 		)
@@
 			)
 		)
+		(property "LCSC" "C53202145"
+			(at 71.12 104.14 0)
+			(effects
+				(font
+					(size 1.27 1.27)
+				)
+				(hide yes)
+			)
+		)
 		(pin "A1"
 		)
@@
 			)
 		)
+		(property "LCSC" "C713185"
+			(at 349.123 85.8774 0)
+			(effects
+				(font
+					(size 1.27 1.27)
+				)
+				(hide yes)
+			)
+		)
 		(pin "+"
 		)
@@
 			)
 		)
+		(property "LCSC" "C53202145"
+			(at 185.42 124.46 0)
+			(effects
+				(font
+					(size 1.27 1.27)
+				)
+				(hide yes)
+			)
+		)
 		(pin "A1"
 		)
@@
 			)
 		)
+		(property "LCSC" "C713185"
+			(at 460.883 85.8774 0)
+			(effects
+				(font
+					(size 1.27 1.27)
+				)
+				(hide yes)
+			)
+		)
 		(pin "+"
 		)
@@
 			)
 		)
+		(property "LCSC" "C53202145"
+			(at 414.02 124.46 0)
+			(effects
+				(font
+					(size 1.27 1.27)
+				)
+				(hide yes)
+			)
+		)
 		(pin "A1"
 		)
@@
 			)
 		)
+		(property "LCSC" "C713185"
+			(at 224.663 85.8774 0)
+			(effects
+				(font
+					(size 1.27 1.27)
+				)
+				(hide yes)
+			)
+		)
 		(pin "+"
 		)
@@
 			)
 		)
+		(property "LCSC" "C713185"
+			(at 51.943 164.6174 0)
+			(effects
+				(font
+					(size 1.27 1.27)
+				)
+				(hide yes)
+			)
+		)
 		(pin "+"
 		)
@@
 			)
 		)
+		(property "LCSC" "C713185"
+			(at 341.503 85.8774 0)
+			(effects
+				(font
+					(size 1.27 1.27)
+				)
+				(hide yes)
+			)
+		)
 		(pin "+"
 		)
@@
 			)
 		)
+		(property "LCSC" "C6332196"
+			(at 148.59 220.98 0)
+			(effects
+				(font
+					(size 1.27 1.27)
+				)
+				(hide yes)
+			)
+		)
 		(pin "1"
 		)
@@
 			)
 		)
+		(property "LCSC" "C53202145"
+			(at 302.26 124.46 0)
+			(effects
+				(font
+					(size 1.27 1.27)
+				)
+				(hide yes)
+			)
+		)
