File: Board/Shortbus.kicad_sch (KiCad schematic)
At the start: 4 parts

Commit message: layout ubus 2.1a
Parts:
- added JP18, JP19: JP1E, csa_ultrabus_v2:JP1, symbol csa_ultrabus_v2-eagle-import:JP1E
Connections:
- net VCC: now also JP18.2, JP19.2; no longer U$2.C1 (VCC), U$2.C16 (VCC2)
- net VCC33: no longer U$2.B14 (VCC33)
- new net: JP18.1, JP19.1, U$2.C1 (VCC), U$2.C16 (VCC2)
Other:
- note added: "CS/A65 Ultra BUS 2.1A"
- note removed: "CS/A65 Ultra BUS 2.0B"
- moved on the sheet: C24

Commit message: candidate
Parts:
- C23, C24: LCSC (none) -> C713185
- JP18, JP19: LCSC (none) -> C7494857
- U$1: LCSC (none) -> C5377847
- U$2: LCSC (none) -> C5173369
Changed lines of the file:
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@@
+			)
+		)
+		(property "LCSC" "C7494857"
+			(at 298.45 73.025 0)
+			(effects
+				(font
+					(size 1.27 1.27)
+				)
+				(hide yes)
 			)
 		)
@@
 			)
 		)
+		(property "LCSC" "C5173369"
+			(at 269.24 109.22 0)
+			(effects
+				(font
+					(size 1.27 1.27)
+				)
+				(hide yes)
+			)
+		)
 		(pin "A1"
 		)
@@
 			)
 		)
+		(property "LCSC" "C5377847"
+			(at 180.34 109.22 0)
+			(effects
+				(font
+					(size 1.27 1.27)
+				)
+				(hide yes)
+			)
+		)
 		(pin "A1"
 		)
@@
 			)
 		)
+		(property "LCSC" "C713185"
+			(at 204.343 70.6374 0)
+			(effects
+				(font
+					(size 1.27 1.27)
+				)
+				(hide yes)
+			)
+		)
 		(pin "+"
 		)
@@
 			)
 		)
+		(property "LCSC" "C7494857"
+			(at 298.45 64.77 0)
+			(effects
+				(font
+					(size 1.27 1.27)
+				)
+				(hide yes)
+			)
+		)
 		(pin "1"
 		)
@@
 			)
 		)
+		(property "LCSC" "C713185"
+			(at 316.738 70.6374 0)
+			(effects
+				(font
+					(size 1.27 1.27)
+				)
+				(hide yes)
+			)
+		)
