File: pwrtest/usbpd-adapter.kicad_sch (KiCad schematic)
At the start: 9 parts, among them J3 USB_C_Receptacle_USB2.0_16P, U9 CH224K

Commit message: update usb-c pwr adapter with mounting holes
Parts:
- added H1, H2, H3, H4: MountingHole, MountingHole:MountingHole_3.2mm_M3_DIN965, symbol Mechanical:MountingHole
- C8: LCSC C33546014 -> C13585
- R29: LCSC (none) -> C5886053
Other:
- note added: "USB-C-PWR-V1.4A-20260909"
- note removed: "USB-C-PWR-V1.3A-20260830"
